File: hardware/QuectoDrive.kicad_sch (KiCad schematic)
At the start: 27 parts, among them U1 SPX3819M5-L-1-8, U2 ATtiny1616-M, U3 DRV8837, U4 DRV8837

Commit message: Board Rev 2
Parts:
- added TP13, TP14, TP7: PROG, TestPoint:TestPoint_Pad_D1.5mm, symbol Connector:TestPoint
- TP5: footprint TestPoint:TestPoint_Pad_D1.0mm -> TestPoint:TestPoint_Pad_D1.5mm
Connections:
- net GND: now also TP13.1; no longer D1.1 (K), U2.10 (PB4), U2.11 (PB3)
- net IO_2: now also U2.16 (PC1); no longer U2.2 (PA3)
- net MOT_2B: now also U2.7 (PA6); no longer U2.9 (PB5)
- net at R1.2: now also D1.1 (K); no longer D1.2 (A)
- net DEBUG_TX: now reaches U2.20 (PA1)
- net DEBUG_TX: now also TP14.1
- net +3V3 renamed +3.3V
- net +3.3V: now also D1.2 (A), TP7.1
- no-connect marks 7 -> 8
Other:
- note added: "TCA WO4"
- note added: "TCD0 WOC"
- note added: "TCD0 WOD"
- note added: "USART0 TXD"
- note removed: "TCB0 WO"
- note removed: "TCB1 WO"
- moved on the sheet: C1, C2, C6, C9, D1, TP11, TP12, TP5, U1, U4
